File: sot23-prog-v1.kicad_sch (KiCad schematic)
At the start: 12 parts, among them J1 Conn_02x05_Odd_Even, J2 Conn_02x06_Row_Letter_First, J3 Conn_02x03_Counter_Clockwise

Commit message: schematic: added comment
Other:
- note added: "Ribbon cable connects to the Azoteq CT210 programmer."
- company: (none) -> by Till Straumann
Changed lines of the file:
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@@
 (kicad_sch (version 20230121) (generator eeschema)
   (paper "A4")
+  (title_block
+    (company "by Till Straumann")
+    (comment 1 "License: public domain")
+  )
   (junction (at 64.77 116.84) (diameter 0) (color 0 0 0 0)
   )
@@
     (effects (font (size 1.27 1.27)) (justify left bottom))
   )
+  (text "Ribbon cable connects to the\nAzoteq CT210 programmer."
+    (at 24.13 107.95 0)
+    (effects (font (size 1.27 1.27)) (justify left bottom))
+  )
